File: Dual_Transistor_AMP.sch (KiCad schematic (older format))
At the start: 14 parts, among them J1 Screw_Terminal_01x02, J2 Screw_Terminal_01x02, Q1 BC548, Q2 BC548

Commit message: Add files via upload
Parts:
- added J3: Screw_Terminal_01x02, TerminalBlock_4Ucon:TerminalBlock_4Ucon_1x02_P3.50mm_Horizontal, symbol Connector:Screw_Terminal_01x02
Connections:
- net +9V: now also J3.1 (Pin_1)
- net GND: now also J3.2 (Pin_2)
Changed lines of the file:
@@
-$EndComp
-$Comp
-L power:PWR_FLAG #FLG01
-U 1 1 61789888
-P 4400 2700
-F 0 "#FLG01" H 4400 2775 50  0001 C CNN
-F 1 "PWR_FLAG" H 4400 2873 50  0000 C CNN
-F 2 "" H 4400 2700 50  0001 C CNN
-F 3 "~" H 4400 2700 50  0001 C CNN
-	1    4400 2700
-	1    0    0    -1
 $EndComp
 $Comp
 L power:+9V #PWR03
 U 1 1 61789AE1
-P 4700 2700
-F 0 "#PWR03" H 4700 2550 50  0001 C CNN
-F 1 "+9V" H 4715 2873 50  0000 C CNN
-F 2 "" H 4700 2700 50  0001 C CNN
-F 3 "" H 4700 2700 50  0001 C CNN
-	1    4700 2700
+P 4800 2300
+F 0 "#PWR03" H 4800 2150 50  0001 C CNN
+F 1 "+9V" H 4815 2473 50  0000 C CNN
+F 2 "" H 4800 2300 50  0001 C CNN
+F 3 "" H 4800 2300 50  0001 C CNN
+	1    4800 2300
 	1    0    0    -1
 $EndComp
@@
 $EndComp
 Wire Wire Line
-	4700 2700 4700 2800
-Wire Wire Line
 	4700 2800 4400 2800
 Wire Wire Line
 	4400 2800 4400 2900
+$Comp
+L Connector:Screw_Terminal_01x02 J3
+U 1 1 61A0FBD0
+P 5350 2100
+F 0 "J3" V 5450 2000 50  0000 L CNN
+F 1 "Screw_Terminal_01x02" V 5550 1700 50  0000 L CNN
+F 2 "TerminalBlock_4Ucon:TerminalBlock_4Ucon_1x02_P3.50mm_Horizontal" H 5350 2100 50  0001 C CNN
+F 3 "https://eu.mouser.com/datasheet/2/445/691214110003-1719301.pdf" H 5350 2100 50  0001 C CNN
+	1    5350 2100
+	0    -1   -1   0
+$EndComp
+$Comp
+L power:GND #PWR0101
+U 1 1 61A160EF
+P 5450 2300
+F 0 "#PWR0101" H 5450 2050 50  0001 C CNN
+F 1 "GND" H 5455 2127 50  0000 C CNN
+F 2 "" H 5450 2300 50  0001 C CNN
+F 3 "" H 5450 2300 50  0001 C CNN
+	1    5450 2300
+	1    0    0    -1
+$EndComp
+$Comp
+L power:PWR_FLAG #FLG0101
+U 1 1 61A16C42
+P 5100 2300
+F 0 "#FLG0101" H 5100 2375 50  0001 C CNN
+F 1 "PWR_FLAG" H 5100 2473 50  0000 C CNN
+F 2 "" H 5100 2300 50  0001 C CNN
+F 3 "~" H 5100 2300 50  0001 C CNN
+	1    5100 2300
+	1    0    0    -1
+$EndComp
 Wire Wire Line
-	4400 2700 4400 2800
-Connection ~ 4400 2800
+	4800 2300 5100 2300
+Connection ~ 5100 2300
+Wire Wire Line
+	5100 2300 5350 2300
+Wire Wire Line
+	4800 2300 4700 2300
+Wire Wire Line
+	4700 2300 4700 2800
+Connection ~ 4800 2300
 $EndSCHEMATC
